Commit message: Add files via upload
needs skid steer / inertias

File: basic_mobile_robot/models/basic_mobile_bot_v1.urdf (robot description, URDF)
Before this commit: robot basic_mobile_bot, 5 links, 4 joints
Joints:
- joint base_joint: child base_link -> base_footprint ; parent base_footprint -> base_link

File: basic_mobile_robot/models/basic_mobile_bot_v2.urdf (robot description, URDF)
Before this commit: robot basic_mobile_bot, 6 links, 5 joints
Links:
- removed link front_caster
- added link cage_link; collision mesh filename=package://basic_mobile_robot/meshes/cage.stl; visual mesh filename=package://basic_mobile_robot/meshes/cage.stl
- link base_link: geometry collision box size=${base_length} ${base_width} ${base_height}; visual mesh filename=package://basic_mobile_robot/meshes/chassis.stl
- link lidar_link: geometry collision mesh filename=package://basic_mobile_robot/meshes/rplidar_s1.stl; visual mesh filename=package://basic_mobile_robot/meshes/rplidar_s1.stl
Joints:
- removed joint caster_joint
- added joint cage_joint: type fixed, parent base_link, child cage_link, origin xyz=0.0 0.0 .119 rpy=0 0 0
- joint base_joint: child base_link -> base_footprint; origin xyz=0.0 0.0 ${(wheel_radius+wheel_zoff)} rpy=0 0 0 -> xyz=0.0 0.0 ${(wheel_radius-wheel_z_offset)} rpy=0 0 0; parent base_footprint -> base_link
- joint lidar_joint: origin xyz=0.215 0 0.13 rpy=0 0 0 -> xyz=0.3885 0 0.192 rpy=0 0 0
